File: _autosave-Fallyx_EVK-RevA.kicad_pcb (KiCad board)
At the start: 4 copper layers, 60.3 x 55 mm, 76 parts, among them IC1 NCH-RSL10-101S51-ACG, J1 Conn_01x05_Pin, J10 MTSW-101-X-X-D-X, J11 Conn_01x01_Pin, J13 Conn_02x20_Odd_Even, J14 Conn_02x18_Odd_Even, J2 Conn_01x06_Pin, J3 Conn_01x06_Pin, J4 Conn_01x08_Pin, J5 MTSW-101-X-X-D-X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

Commit message: review edits
Parts:
- removed J10: MTSW-101-X-X-D-X, MTSW-101-X-X-D-X:SAMTEC_MTSW-101-X-X-D-X
- removed J13: Conn_02x20_Odd_Even, Connector_PinHeader_2.54mm:PinHeader_2x20_P2.54mm_Vertical
