File: Fallyx_EVK-RevA.kicad_pcb (KiCad board)
At the start: 4 copper layers, 60.3 x 55 mm, 76 parts, among them IC1 NCH-RSL10-101S51-ACG, J1 Conn_01x05_Pin, J10 MTSW-101-X-X-D-X, J11 Conn_01x01_Pin, J13 Conn_02x20_Odd_Even, J14 Conn_02x18_Odd_Even, J2 Conn_01x06_Pin, J3 Conn_01x06_Pin, J4 Conn_01x08_Pin, J5 MTSW-101-X-X-D-X, J6 USB_C_6P, U1 XC9236F08CER-G, U2 ILPS22QSTR, U3 BMI270, U4 STM32L431VCIx, U5 MX25R3235FZNxx0, U6 MCP73831T-2ACI_OT, U7 BQ27421YZFR-G1A, X1 8MHz, X2 32.768kHz

Commit message: Updated for new BLE modules
Parts:
- removed C10: 10pF, Capacitor_SMD:C_0402_1005Metric
- removed C11, C13: 1uF, Capacitor_SMD:C_0402_1005Metric
- removed C12: 0.1uF, Capacitor_SMD:C_0402_1005Metric
- removed C9: 22nuF, Capacitor_SMD:C_0402_1005Metric
- removed J10: MTSW-101-X-X-D-X, MTSW-101-X-X-D-X:SAMTEC_MTSW-101-X-X-D-X
- removed J14: Conn_02x18_Odd_Even, Connector_PinHeader_2.54mm:PinHeader_2x18_P2.54mm_Vertical
- removed R11: 10k, Resistor_SMD:R_0402_1005Metric
- removed R12: 1k, Resistor_SMD:R_0402_1005Metric
- removed R13: 0R, Resistor_SMD:R_0805_2012Metric
- added C33: 2.2uF, Capacitor_SMD:C_0603_1608Metric, F.Cu at (131.6, 107.8)
- added C34: 22uF, Capacitor_SMD:C_0603_1608Metric, F.Cu at (155.8, 67.0)
- added C35: 1uF, Capacitor_SMD:C_0402_1005Metric, F.Cu at (131.8, 69.1)
- added C36: 0.1uF, Capacitor_SMD:C_0402_1005Metric, F.Cu at (130.7, 75.4)
- added C37: 1uF, Capacitor_SMD:C_0402_1005Metric, F.Cu at (131.8, 75.4)
- added C38: 22nF, Capacitor_SMD:C_0402_1005Metric, F.Cu at (132.6, 82.9)
- added C39: 10pF, Capacitor_SMD:C_0402_1005Metric, F.Cu at (132.6, 80.7)
- added C40: 22uF, Capacitor_SMD:C_0603_1608Metric, F.Cu at (174.8, 94.2)
- added C41: 4.7uF, Capacitor_SMD:C_0603_1608Metric, F.Cu at (170.1, 118.8)
- added C42: 1.2pF, Capacitor_SMD:C_0402_1005Metric, F.Cu at (152.8, 100.7)
- added C43: 1.2pF, Capacitor_SMD:C_0402_1005Metric, F.Cu at (152.8, 103.9)
- added C44: 4.7uF, Capacitor_SMD:C_0603_1608Metric, F.Cu at (153.6, 89.9)
- added C45: 150pF, Capacitor_SMD:C_0603_1608Metric, F.Cu at (158.3, 86.6)
- added C46: 10uF, Capacitor_SMD:C_0805_2012Metric, F.Cu at (160.9, 85.7)
- added D1: GREEN, LED_SMD:LED_0603_1608Metric, F.Cu at (113.7, 86.2)
- added D2: RED, LED_SMD:LED_0603_1608Metric, F.Cu at (125.1, 85.8)
- added D3: AMBER, LED_SMD:LED_0603_1608Metric, F.Cu at (120.7, 85.8)
- added D4: APG0603SURC-TT, APG0603SURC-TT:LED_APG0603SURC-TT, F.Cu at (126.7, 78.3)
- added D5: RB521S30T1G, RB521S30T1G:DIOM168X70N, F.Cu at (117.6, 82.8)
- added D6: APG0603SURC-TT, APG0603SURC-TT:LED_APG0603SURC-TT, F.Cu at (155.8, 103.8)
- added FB2: 600R/0.7A, Resistor_SMD:R_0402_1005Metric, F.Cu at (130.7, 77.8)
- added J12: Conn_02x20_Odd_Even, Connector_PinHeader_2.54mm:PinHeader_2x20_P2.54mm_Vertical, F.Cu at (114.0, 96.6)
- added J7: Conn_01x01_Pin, Connector_PinHeader_2.54mm:PinHeader_1x01_P2.54mm_Vertical, F.Cu at (117.2, 88.6)
- added J8: Conn_01x01_Pin, Connector_PinHeader_2.54mm:PinHeader_1x01_P2.54mm_Vertical, F.Cu at (124.0, 88.6)
- added J9: U.FL-R-SMT-1_80_, U.FL-R-SMT-1_80_:HIROSE_U.FL-R-SMT-1_80_, F.Cu at (156.2, 101.3)
- added L2: 3.3nH, Inductor_SMD:L_0402_1005Metric, F.Cu at (152.3, 102.3)
- added L3: 4.7uH, NR3015T4R7M:IND_TAIYO_NR3015_TAY, F.Cu at (161.0, 89.6)
- added Q1: 2SK3018T106H71, Package_TO_SOT_SMD:SOT-323_SC-70, F.Cu at (120.6, 88.5)
- added Q2: LMBT3904WT1G, Package_TO_SOT_SMD:SOT-23, F.Cu at (127.7, 88.8)
- added R19: 100k, Resistor_SMD:R_0402_1005Metric, F.Cu at (158.2, 80.3)
- added R20: 1k, Resistor_SMD:R_0402_1005Metric, F.Cu at (125.3, 77.8)
- added R21: 100R, Resistor_SMD:R_0402_1005Metric, F.Cu at (118.0, 91.5)
- added R22: 10k, Resistor_SMD:R_0402_1005Metric, F.Cu at (120.2, 91.5)
- added R23: 10k, Resistor_SMD:R_0402_1005Metric, F.Cu at (127.2, 91.5)
- added R24: 100R, Resistor_SMD:R_0402_1005Metric, F.Cu at (118.5, 85.5)
- added R25: 1k, Resistor_SMD:R_0402_1005Metric, F.Cu at (122.9, 85.5)
- added R26: 1k, Resistor_SMD:R_0402_1005Metric, F.Cu at (110.8, 86.2)
- added R27: 0R, Resistor_SMD:R_0805_2012Metric, F.Cu at (130.2, 68.3)
- added R28: 10k, Resistor_SMD:R_0402_1005Metric, F.Cu at (137.2, 67.0)
- added R29: 1k, Resistor_SMD:R_0402_1005Metric, F.Cu at (132.6, 81.8)
- added R30: 4.7k, Resistor_SMD:R_0402_1005Metric, F.Cu at (171.9, 112.2)
- added R31: 320k, Resistor_SMD:R_0402_1005Metric, F.Cu at (158.3, 85.3)
- added R32: 150k, Resistor_SMD:R_0402_1005Metric, F.Cu at (158.3, 84.3)
- added U10: XC9236F08CER-G, XC9236F:XC9236F08CERG, F.Cu at (156.6, 89.4)
- added U8: RN4871-I/RM140, RF_Module:Microchip_RN4871, F.Cu at (169.1, 86.6)
- added U9: BM70BLE01FC2-0B04AA, BM70BLE01FC2:BM70BLE01FC2_MCH, F.Cu at (158.7, 111.5)
- J13: value Conn_02x20_Odd_Even -> Conn_01x09; footprint Connector_PinHeader_2.54mm:PinHeader_2x20_P2.54mm_Vertical -> Connector_PinHeader_2.54mm:PinHeader_1x09_P2.54mm_Vertical
- U4: value STM32L431VCIx -> STM32L431CBT6; footprint Package_BGA:UFBGA-100_7x7mm_Layout12x12_P0.5mm -> STM32L431CBT6:LQFP-48
- moved J13 30.6 mm to (174.7, 97.4)
- moved C14 6.61 mm to (144.9, 67.8), turned to 90 degrees
- moved C15 5.81 mm to (140.7, 79.0), turned to 180 degrees
- moved IC1 4.36 mm to (159.3, 72.6)
- moved J4 4.36 mm to (151.8, 68.3)
- moved C27 4.36 mm to (159.2, 77.5)
- moved C28 4.36 mm to (157.2, 77.7)
- moved R15 4.36 mm to (158.8, 78.8)
- moved C21 2.81 mm to (144.7, 70.5), turned to -90 degrees
- moved J11 1.75 mm to (145.1, 101.8)
- moved R18 1.75 mm to (144.9, 117.7)
- moved S1 1.75 mm to (145.0, 110.7)
- moved C23 1.60 mm to (132.6, 79.6)
- moved C26 1.60 mm to (134.6, 79.6)
- moved U5 1.60 mm to (138.5, 83.7)
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Connections:
- J13 pad 1: unconnected-(J13-Pin_1-Pad1) -> BLE2_VDD
- J13 pad 2: unconnected-(J13-Pin_2-Pad2) -> GND
- J13 pad 3: unconnected-(J13-Pin_3-Pad3) -> BLE2_CTS
- J13 pad 4: unconnected-(J13-Pin_4-Pad4) -> BLE2_P3_6
- J13 pad 5: unconnected-(J13-Pin_5-Pad5) -> BLE2_TX
- J13 pad 6: unconnected-(J13-Pin_6-Pad6) -> BLE2_RX
- J13 pad 7: unconnected-(J13-Pin_7-Pad7) -> BLE2_RST_N
- J13 pad 8: unconnected-(J13-Pin_8-Pad8) -> BLE2_P2_0
- J13 pad 9: unconnected-(J13-Pin_9-Pad9) -> BLE2_P2_7
- U7 pad A2: I2C2_SDA -> BLE_UART_TX
- U7 pad A3: I2C2_SCL -> BLE_UART_RX
Routing:
- net BLE2_VDD: track 0.00 -> 95.9 mm, vias 0 -> 5
- net JTMS_SWCLK: track 0.00 -> 64.1 mm, vias 0 -> 1
- net V_IN: track 14.6 -> 78.2 mm
- net BLE2_P2_7: track 0.00 -> 63.1 mm, vias 0 -> 1
- net GND: track 112.0 -> 175.0 mm, vias 34 -> 53
- net BLE_UART_RX: track 9.05 -> 71.2 mm, vias 0 -> 2
- net BLE_UART_TX: track 6.04 -> 65.4 mm, vias 0 -> 2
- net GPOUT: track 19.4 -> 77.3 mm
- net BLE2_P2_0: track 0.00 -> 56.2 mm, vias 0 -> 1
- net PB7: track 0.00 -> 52.4 mm, vias 0 -> 1
- net PB6: track 0.00 -> 48.3 mm, vias 0 -> 1
- net PB5: track 0.00 -> 47.9 mm, vias 0 -> 1
- net BLE_WAKE: track 16.7 -> 60.6 mm, vias 0 -> 1
- net BLE2_P3_6: track 0.00 -> 42.0 mm, vias 0 -> 1
- net BLE_RESET: track 20.3 -> 61.7 mm, vias 2 -> 3
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- added copper zone on F.Cu, net /Fallyx_EVK_6/LX2.5
- added copper zone on F.Cu, net BLE2_VDD
- added copper zone on B.Cu, net GND
- added copper zone on F.Cu, net GND
- added copper zone on F.Cu, net Net-(U10-VOUT(FB))
Other:
- board size 60.3 x 55 mm -> 77.3 x 55 mm
- board text added: "BYPASS"
