File: Fallyx_EVK_3.kicad_sch (KiCad schematic)
At the start: 8 parts, among them J2 Conn_01x06_Pin, J3 Conn_01x06_Pin, U3 BMI270

Commit message: continued design work
Parts:
- added J10: MTSW-101-X-X-D-X, MTSW-101-X-X-D-X:SAMTEC_MTSW-101-X-X-D-X, symbol MTSW-101-X-X-D-X:MTSW-101-X-X-D-X
- J2, J3: footprint (none) -> Connector_PinHeader_2.54mm:PinHeader_1x06_P2.54mm_Vertical
Other:
- note added: "FORCE RESISTOR"
- note added: "TACTILE BUTTON"
Changed lines of the file:
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@@
+		)
+	)
+	(text "FORCE RESISTOR"
+		(exclude_from_sim no)
+		(at 66.294 111.76 0)
+		(effects
+			(font
+				(size 2.54 2.54)
+				(thickness 0.508)
+				(bold yes)
+			)
 		)
 	)
@@
 			(font
 				(size 1.27 1.27)
+			)
+		)
+	)
+	(text "TACTILE BUTTON"
+		(exclude_from_sim no)
+		(at 229.108 111.76 0)
+		(effects
+			(font
+				(size 2.54 2.54)
+				(thickness 0.508)
+				(bold yes)
 			)
 		)
@@
 	)
 	(symbol
+		(lib_id "MTSW-101-X-X-D-X:MTSW-101-X-X-D-X")
+		(at 38.1 139.7 90)
+		(unit 1)
+		(exclude_from_sim no)
+		(in_bom yes)
+		(on_board yes)
+		(dnp no)
+		(fields_autoplaced yes)
+		(property "Reference" "J10"
+			(at 41.91 139.6999 90)
+			(effects
+				(font
+					(size 1.27 1.27)
+				)
+				(justify right)
+			)
+		)
+		(property "Value" "MTSW-101-X-X-D-X"
+			(at 41.91 140.9699 90)
+			(effects
+				(font
+					(size 1.27 1.27)
+				)
+				(justify right)
+				(hide yes)
+			)
+		)
+		(property "Footprint" "MTSW-101-X-X-D-X:SAMTEC_MTSW-101-X-X-D-X"
+			(at 38.1 139.7 0)
+			(effects
+				(font
+					(size 1.27 1.27)
+				)
+				(justify bottom)
+				(hide yes)
+			)
+		)
+		(property "Datasheet" ""
+			(at 38.1 139.7 0)
+			(effects
+				(font
+					(size 1.27 1.27)
+				)
+				(hide yes)
+			)
+		)
+		(property "Description" ""
+			(at 38.1 139.7 0)
+			(effects
+				(font
+					(size 1.27 1.27)
+				)
+				(hide yes)
+			)
+		)
+		(property "MF" "Samtec"
+			(at 38.1 139.7 0)
+			(effects
+				(font
+					(size 1.27 1.27)
+				)
+				(justify bottom)
+				(hide yes)
+			)
+		)
+		(property "Description_1" "\n                        \n                            Connector Header Through Hole 2 position\n                        \n"
+			(at 38.1 139.7 0)
+			(effects
+				(font
+					(size 1.27 1.27)
+				)
+				(justify bottom)
+				(hide yes)
+			)
+		)
+		(property "Package" "None"
+			(at 38.1 139.7 0)
+			(effects
+				(font
+					(size 1.27 1.27)
+				)
+				(justify bottom)
+				(hide yes)
+			)
+		)
+		(property "Price" "None"
+			(at 38.1 139.7 0)
+			(effects
+				(font
+					(size 1.27 1.27)
+				)
+				(justify bottom)
+				(hide yes)
+			)
+		)
+		(property "Check_prices" "https://www.snapeda.com/parts/MTSW-101-08-S-D-318/Samtec/view-part/?ref=eda"
+			(at 38.1 139.7 0)
+			(effects
+				(font
+					(size 1.27 1.27)
+				)
+				(justify bottom)
+				(hide yes)
+			)
+		)
+		(property "STANDARD" "Manufacturer recommendations"
+			(at 38.1 139.7 0)
+			(effects
+				(font
+					(size 1.27 1.27)
+				)
+				(justify bottom)
+				(hide yes)
+			)
+		)
+		(property "PARTREV" "A"
+			(at 38.1 139.7 0)
+			(effects
+				(font
+					(size 1.27 1.27)
+				)
+				(justify bottom)
+				(hide yes)
+			)
+		)
+		(property "SnapEDA_Link" "https://www.snapeda.com/parts/MTSW-101-08-S-D-318/Samtec/view-part/?ref=snap"
+			(at 38.1 139.7 0)
+			(effects
+				(font
+					(size 1.27 1.27)
+				)
+				(justify bottom)
+				(hide yes)
+			)
+		)
+		(property "MP" "MTSW-101-08-S-D-318"
+			(at 38.1 139.7 0)
+			(effects
+				(font
+					(size 1.27 1.27)
+				)
+				(justify bottom)
+				(hide yes)
+			)
+		)
+		(property "Availability" "In Stock"
+			(at 38.1 139.7 0)
+			(effects
+				(font
+					(size 1.27 1.27)
+				)
+				(justify bottom)
+				(hide yes)
+			)
+		)
+		(property "MANUFACTURER" "Samtec"
+			(at 38.1 139.7 0)
+			(effects
+				(font
+					(size 1.27 1.27)
+				)
+				(justify bottom)
+				(hide yes)
+			)
+		)
+		(pin "02"
+		)
+		(pin "01"
+		)
+		(instances
+			(project "Fallyx_EVK-RevA"
+				(path "/c9ecf77f-e2c2-430e-a6fe-72307adaa202/efa7fa42-336a-4c4b-a853-30b1840ce713"
+					(reference "J10")
+					(unit 1)
+				)
+			)
+		)
+	)
+	(symbol
 		(lib_id "power:GND")
 		(at 248.92 62.23 0)
@@
 			)
 		)
-		(property "Footprint" ""
+		(property "Footprint" "Connector_PinHeader_2.54mm:PinHeader_1x06_P2.54mm_Vertical"
 			(at 260.35 81.28 0)
 			(effects
@@
 			)
 		)
-		(property "Footprint" ""
+		(property "Footprint" "Connector_PinHeader_2.54mm:PinHeader_1x06_P2.54mm_Vertical"
 			(at 259.08 49.53 0)
 			(effects

Commit message: review edits
Parts:
- added C33: 2.2uF, Capacitor_SMD:C_0603_1608Metric, symbol Device:C_Small
- added J11: Conn_01x01_Pin, Connector_PinHeader_2.54mm:PinHeader_1x01_P2.54mm_Vertical, symbol Connector:Conn_01x01_Pin
- added R18: 10k, Resistor_SMD:R_0402_1005Metric, symbol Device:R_US
- added S1: TS04-66-50-BK-100-SMT, TS04-66-50-BK-100-SMT:SW_TS04-66-50-BK-100-SMT, symbol TS04-66-50-BK-100-SMT:TS04-66-50-BK-100-SMT
Connections:
- net 1V8: now also C33.1, R18.1
- net GND: now also C33.2, S1.4
- new net: R18.2, S1.3
- new net SW1_OUTPUT: J11.1 (Pin_1), S1.1
Other:
- moved on the sheet: C7, C8, R8, R9

Commit message: Updated for new BLE modules
Changed lines of the file:
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@@
+		)
+	)
+	(polyline
+		(pts
+			(xy 25.4 127) (xy 50.8 152.4)
+		)
+		(stroke
+			(width 1.27)
+			(type default)
+			(color 255 0 17 1)
 		)
 	)
