File: Fallyx_EVK_5.kicad_sch (KiCad schematic)
At the start: 5 parts, among them IC1 NCH-RSL10-101S51-ACG, J4 Conn_01x08_Pin

Commit message: review edits
Parts:
- added C34: 22uF, Capacitor_SMD:C_0603_1608Metric, symbol Device:C
- added R19: 100k, Resistor_SMD:R_0402_1005Metric, symbol Device:R_US
- C27: footprint (none) -> Capacitor_SMD:C_0603_1608Metric
- C28: footprint (none) -> Capacitor_SMD:C_0402_1005Metric
- R15: footprint (none) -> Resistor_SMD:R_0402_1005Metric
Connections:
- net 1V8: now also C34.1
- net BLE_WAKE: now also R19.2
- net GND: now also C34.2, R19.1
Other:
- note added: "DNP"
- moved on the sheet: C27, C28, J4

Commit message: Updated for new BLE modules
Parts:
- added C40: 22uF, Capacitor_SMD:C_0603_1608Metric, symbol Device:C
- added C41: 4.7uF, Capacitor_SMD:C_0603_1608Metric, symbol Device:C
- added C42, C43: 1.2pF, Capacitor_SMD:C_0402_1005Metric, symbol Device:C
- added D6: APG0603SURC-TT, APG0603SURC-TT:LED_APG0603SURC-TT, symbol APG0603SURC-TT:APG0603SURC-TT
- added IC2: BGM111A256V21R, BGM111A256:BGM111A256V21R, symbol BGM111A256V21R:BGM111A256V21R
- added J13: Conn_01x09, Connector_PinHeader_2.54mm:PinHeader_1x09_P2.54mm_Vertical, symbol Connector_Generic:Conn_01x09
- added J9: U.FL-R-SMT-1_80_, U.FL-R-SMT-1_80_:HIROSE_U.FL-R-SMT-1_80_, symbol U.FL-R-SMT-1_80_:U.FL-R-SMT-1_80_
- added L2: 3.3nH, Inductor_SMD:L_0402_1005Metric, symbol Device:L_Small
- added R30: 4.7k, Resistor_SMD:R_0402_1005Metric, symbol Device:R_US
- added U8: RN4871-I/RM140, RF_Module:Microchip_RN4871, symbol RN4871:RN4871-I_RM140
- added U9: BM70BLE01FC2-0B04AA, BM70BLE01FC2:BM70BLE01FC2_MCH, symbol BM70BLE01FC2:BM70BLE01FC2-0B04AA
Connections:
- net GND: now also C40.2, C41.2, C42.2, C43.2, IC2.1 (GND_1), IC2.12 (GND_2), IC2.20 (GND_3), IC2.31 (GND_4), J13.2 (Pin_2), J9.G1, J9.G2, U8.13 (GND), U8.2 (GND), U9.1 (GND), U9.29 (GND)
- new net: C42.1, J9.SIG, L2.2
- new net BLE2_ANT: C43.1, L2.1, U9.30 (BT_RF)
- new net BLE2_CTS: IC2.8 (PA3), J13.3 (Pin_3), U8.11 (P0_0), U9.13 (P0_0/CTS)
- new net BLE2_P0_2: D6.1, U8.12 (P0_2), U9.28 (P0_2/LED)
- new net BLE2_P1_2: U8.3 (P1_2), U9.11 (P1_2/SCL)
- new net BLE2_P1_3: U8.4 (P1_3), U9.12 (P1_3/SDA)
- new net BLE2_P1_6: U8.6 (P1_6)
- new net BLE2_P1_7: U8.5 (P1_7)
- new net BLE2_P2_0: J13.8 (Pin_8), U8.16 (P2_0), U9.16 (P2_0/MODE)
- new net BLE2_P2_7: J13.9 (Pin_9), U8.15 (P2_7), U9.9 (P2_7/TX_IND)
- new net BLE2_P3_6: IC2.7 (PA2), J13.4 (Pin_4), U8.9 (P3_6), U9.15 (P3_6/RTS)
- new net BLE2_RST: IC2.30 (RESETN)
- new net BLE2_RST_N: J13.7 (Pin_7), R30.1, U8.10 (RST_N), U9.18 (NC), U9.19 (RST_N)
- new net BLE2_RX: IC2.5 (PA0), J13.6 (Pin_6), U8.7 (UART_RX), U9.20 (HCI_RXD)
- new net BLE2_SWCLK: IC2.21 (PF0)
- new net BLE2_SWDIO: IC2.22 (PF1)
- new net BLE2_TX: IC2.6 (PA1), J13.5 (Pin_5), U8.8 (UART_TX), U9.21 (HCI_TXD)
- new net BLE2_VDD: C40.1, C41.1, D6.2, IC2.29 (VDD), J13.1 (Pin_1), R30.2, U8.14 (VBAT), U9.2 (VBAT)
- no-connect marks 19 -> 55
Other:
- note added: "BLE MODULE ALT"
- moved on the sheet: J4

Commit message: Final Routing and export for EVK
Other:
- note added: "Z0 = 50 Ohm. 0.18mm Trace @ 0.1h dielectric"
Changed lines of the file:
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@@
+		)
+	)
+	(text "Z0 = 50 Ohm.\n0.18mm Trace @ 0.1h dielectric"
+		(exclude_from_sim no)
+		(at 249.936 151.892 0)
+		(effects
+			(font
+				(size 1.27 1.27)
+			)
+			(justify left)
 		)
 	)
